Commit message: initial position of g0 setup

File: source/g0_robot_lab/g0_robot_lab/assets/robots/g0/urdf/g0.urdf (robot description, URDF)
Before this commit: robot g0, 23 links, 22 joints
Links:
- link r_shoulder_roll_link: mass 13.0304549688345 -> 0.0467894808715163

Commit message: fix r_shoulder_roll_link and torso_link problem

File: source/g0_robot_lab/g0_robot_lab/assets/robots/g0/urdf/g0.urdf (robot description, URDF)
Before this commit: robot g0, 23 links, 22 joints
Links:
- link torso_link: mass 0.506639508062444 -> 0.86309508062444

Commit message: urdf changed

File: source/g0_robot_lab/g0_robot_lab/assets/robots/g0/urdf/g0.urdf (robot description, URDF)
Before this commit: robot g0, 23 links, 22 joints
Links:
- link base_link: mass 0.033535963666254 -> 0.033536
- link l_calf_link: mass 0.0287721329481339 -> 0.0287721329481338
- link l_forearm_link: mass 0.0306315007081731 -> 0.030632
- link l_shoulder_pitch_link: mass 0.0379707027827449 -> 0.037971
- link l_shoulder_roll_link: mass 0.0467894808715163 -> 0.046789
- link r_calf_link: mass 0.0287768621501782 -> 0.028776880276565
- link r_forearm_link: mass 0.0306132879831417 -> 0.0306132776535569
- link r_hip_pitch_link: mass 0.0438357899722271 -> 0
- link torso_link: mass 0.86309508062444 -> 0.50948
- link waist_yaw_link: mass 0.0352857278796645 -> 0.035286
Joints:
- joint l_ankle_pitch_joint: axis 0 -1 0 -> 0 1 0
- joint l_ankle_roll_joint: axis -1 0 0 -> 1 0 0
- joint l_elbow_pitch_joint: axis 0 -1 0 -> 0 1 0; limit lower=0 upper=1.2 effort=2 velocity=99 -> lower=-1.2 upper=0 effort=2 velocity=99
- joint l_hip_pitch_joint: origin xyz=1.38715273801726E-05 0.013999999999999 0 rpy=0 0 0 -> xyz=1.3872E-05 0.014 0 rpy=0 0 0
- joint l_hip_roll_joint: axis -1 0 0 -> 1 0 0; limit lower=-0.75 upper=0 effort=2 velocity=99 -> lower=0 upper=0.75 effort=2 velocity=99
- joint l_hip_yaw_joint: axis 0 0 -1 -> 0 0 1
- joint l_knee_pitch_joint: axis 0 -1 0 -> 0 1 0; limit lower=-0.75 upper=0 effort=2 velocity=99 -> lower=0 upper=0.75 effort=2 velocity=99
- joint l_shoulder_pitch_joint: axis 0 -1 0 -> 0 1 0; origin xyz=-0.019982101043914 0.0498030364741947 0.117056041163315 rpy=0 0 0 -> xyz=-0.019982 0.049803 0.11706 rpy=0 0 0
- joint l_shoulder_roll_joint: axis -1 0 0 -> 1 0 0; limit lower=-1.2 upper=0 effort=2 velocity=99 -> lower=0 upper=1.2 effort=2 velocity=99; origin xyz=0.017973963102699 0.0187406777660832 -0.00533315738858231 rpy=0 0 0 -> xyz=0.017974 0.018741 -0.0053332 rpy=0 0 0
- joint l_shoulder_yaw_joint: axis 0 0 -1 -> 0 0 1; origin xyz=-0.0204659061735258 0.00301291158004391 -0.0235668088196405 rpy=0 0 0 -> xyz=-0.020466 0.0030129 -0.023567 rpy=0 0 0
- joint r_ankle_roll_joint: axis -1 0 0 -> 1 0 0
- joint r_hip_pitch_joint: axis 0 -1 0 -> 0 1 0
- joint r_hip_roll_joint: axis -1 0 0 -> 1 0 0; limit lower=0 upper=0.75 effort=2 velocity=99 -> lower=-0.75 upper=0 effort=2 velocity=99
- joint r_hip_yaw_joint: axis 0 0 -1 -> 0 0 1
- joint r_shoulder_roll_joint: axis -1 0 0 -> 1 0 0; limit lower=0 upper=1.2 effort=2 velocity=99 -> lower=-1.2 upper=0 effort=2 velocity=99; origin xyz=0.0179739631027021 -0.018740677766079 -0.00533315738858159 rpy=0 0 0 -> xyz=0.017974 -0.018741 -0.0053332 rpy=0 0 0
- joint r_shoulder_yaw_joint: axis 0 0 -1 -> 0 0 1
- joint waist_roll_joint: axis -1 0 0 -> 1 0 0; origin xyz=0.0199489728093946 -2.77476286030481E-05 0.0145010271906055 rpy=0 0 0 -> xyz=0.01995 -1.3874E-05 0.033929 rpy=0 0 0
- joint waist_yaw_joint: axis 0 0 -1 -> 0 0 1; origin xyz=0 1.38738143016396E-05 0.019428150414191 rpy=0 0 0 -> xyz=0 0 0 rpy=0 0 0

Commit message: sim2sim mujoco

File: source/g0_robot_lab/g0_robot_lab/assets/robots/g0/urdf/g0.urdf (robot description, URDF)
Before this commit: robot g0, 23 links, 22 joints
Links:
- link r_hip_pitch_link: mass 0 -> 0.043836
